File: peripherals.kicad_sch (KiCad schematic)
At the start: 15 parts, among them SW2 BACK_BTN, SW3 EXEC_BTN

Commit message: Modified PCB for Aisler budget tier
Parts:
- SW4: value (none) -> EC11x_Encoder; footprint Rotary_Encoder:RotaryEncoder_Alps_EC11E-Switch_Vertical_H20mm -> (none)
- U6: value (none) -> 25LC256 / GT32L24A180
Changed lines of the file:
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@@
       (effects (font (size 1.27 1.27)) (justify left))
     )
-    (property "Value" "" (id 1) (at 68.0594 124.46 0)
+    (property "Value" "25LC256 / GT32L24A180" (id 1) (at 68.0594 124.46 0)
       (effects (font (size 1.27 1.27)) (justify left))
     )
@@
     (in_bom yes) (on_board yes) (fields_autoplaced)
     (property "Reference" "SW4" (id 0) (at 77.47 77.47 0))
-    (property "Value" "" (id 1) (at 77.47 80.01 0))
-    (property "Footprint" "Rotary_Encoder:RotaryEncoder_Alps_EC11E-Switch_Vertical_H20mm" (id 2) (at 73.66 83.566 0)
-      (effects (font (size 1.27 1.27)) hide)
-    )
+    (property "Value" "EC11x_Encoder" (id 1) (at 77.47 80.01 0))
+    (property "Footprint" "" (id 2) (at 73.66 83.566 0)
+      (effects (font (size 1.27 1.27)) hide)
+    )
