File: tauntek_hat.kicad_pcb (KiCad board)
At the start: 2 copper layers, 161 x 107 mm, 86 parts, among them J1 UPDI, J2 TESTER_PWR, J3 USB-TYPE-C-018, J4 SERIAL_ADAPTER, J5 SERIAL_DB9, J6 TESTER_SERIAL_PORT, Q1 NCE30P12S, Q2 DMG2302U, Q3 DMG2302U, Q4 DMG2302U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

Commit message: Modified PCB for Aisler budget tier
Parts:
- J2: footprint Connector_BarrelJack:BarrelJack_Horizontal -> tauntek-hat:BarrelJack_Horizontal_CircularHoles
- J3: footprint tauntek-hat:USB_C_Receptacle_HRO_TYPE-C-31-M-12_NO_SBU -> tauntek-hat:USB_C_Receptacle_HRO_TYPE-C-31-M-12_NO_SBU_CircularHoles
- SW4: footprint Rotary_Encoder:RotaryEncoder_Alps_EC11E-Switch_Vertical_H20mm -> Rotary_Encoder:RotaryEncoder_Alps_EC11E-Switch_Vertical_H20mm_CircularMountingHoles
- U3: footprint Package_DFN_QFN:QFN-64-1EP_9x9mm_P0.5mm_EP7.15x7.15mm_ThermalVias -> Package_DFN_QFN:QFN-64-1EP_9x9mm_P0.5mm_EP7.15x7.15mm
- moved Q1 0.70 mm to (86.7, 33.1)
- moved J3 0.20 mm to (97.1, 34.5)
Routing:
- net GND: track 63.9 -> 67.7 mm, vias 220 -> 236
- net Net-(J2-Pad1): track 30.8 -> 28.0 mm
- net Net-(D2-Pad2): track 18.4 -> 19.1 mm
- net +9V: track 96.3 -> 97.0 mm
Other:
- outline, holes or cut-outs redrawn
