File: tauntek_hat.kicad_sch (KiCad schematic)
At the start: 36 parts, among them J1 UPDI, J2 TESTER_PWR, Q1 NCE30P12S, Q2 DMG2302U, Q3 DMG2302U, Q4 DMG2302U, SW1 RST_BTN, U1 AMS1117-5.0, U2 AMS1117-3.3, U3 AVR128DB64-IMR

Commit message: Modified PCB for Aisler budget tier
Parts:
- J2: footprint Connector_BarrelJack:BarrelJack_Horizontal -> (none)
- TP1: value (none) -> TestPoint; footprint (none) -> TestPoint:TestPoint_Pad_D1.0mm
- TP2, TP3, TP4: footprint (none) -> TestPoint:TestPoint_Pad_D1.0mm
- U3: footprint Package_DFN_QFN:QFN-64-1EP_9x9mm_P0.5mm_EP7.15x7.15mm_ThermalVias -> (none)
Changed lines of the file:
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@@
       (effects (font (size 1.27 1.27)) (justify left))
     )
-    (property "Value" "" (id 1) (at 269.24 128.2699 90)
-      (effects (font (size 1.27 1.27)) (justify left))
-    )
-    (property "Footprint" "" (id 2) (at 264.16 132.08 0)
+    (property "Value" "TestPoint" (id 1) (at 269.24 128.2699 90)
+      (effects (font (size 1.27 1.27)) (justify left))
+    )
+    (property "Footprint" "TestPoint:TestPoint_Pad_D1.0mm" (id 2) (at 264.16 132.08 0)
       (effects (font (size 1.27 1.27)) hide)
     )
@@
       (effects (font (size 1.27 1.27)) (justify left))
     )
-    (property "Footprint" "Package_DFN_QFN:QFN-64-1EP_9x9mm_P0.5mm_EP7.15x7.15mm_ThermalVias" (id 2) (at 278.13 158.75 0)
+    (property "Footprint" "" (id 2) (at 278.13 158.75 0)
       (effects (font (size 1.27 1.27)) hide)
     )
@@
       (effects (font (size 1.27 1.27)) (justify right))
     )
-    (property "Footprint" "Connector_BarrelJack:BarrelJack_Horizontal" (id 2) (at 92.71 83.566 0)
+    (property "Footprint" "" (id 2) (at 92.71 83.566 0)
       (effects (font (size 1.27 1.27)) hide)
     )
@@
       (effects (font (size 1.27 1.27)) (justify left))
     )
-    (property "Footprint" "" (id 2) (at 264.16 142.24 0)
+    (property "Footprint" "TestPoint:TestPoint_Pad_D1.0mm" (id 2) (at 264.16 142.24 0)
       (effects (font (size 1.27 1.27)) hide)
     )
@@
       (effects (font (size 1.27 1.27)) (justify left))
     )
-    (property "Footprint" "" (id 2) (at 264.16 137.16 0)
+    (property "Footprint" "TestPoint:TestPoint_Pad_D1.0mm" (id 2) (at 264.16 137.16 0)
       (effects (font (size 1.27 1.27)) hide)
     )
@@
     (property "Reference" "TP4" (id 0) (at 194.31 135.89 90))
     (property "Value" "TestPoint" (id 1) (at 196.85 138.43 90))
-    (property "Footprint" "" (id 2) (at 207.01 142.24 0)
+    (property "Footprint" "TestPoint:TestPoint_Pad_D1.0mm" (id 2) (at 207.01 142.24 0)
       (effects (font (size 1.27 1.27)) hide)
     )
@@
     )
     (path "/a2b9a962-6d97-4b01-b4cd-aaff49f4dfe6"
-      (reference "J2") (unit 1) (value "TESTER_PWR") (footprint "Connector_BarrelJack:BarrelJack_Horizontal")
+      (reference "J2") (unit 1) (value "TESTER_PWR") (footprint "tauntek-hat:BarrelJack_Horizontal_CircularHoles")
     )
     (path "/e10271d7-3f19-468d-ac2e-d112f94b8b42/e14aef9d-bcb2-4f21-943c-230b7e6ba0ed"
-      (reference "J3") (unit 1) (value "USB-TYPE-C-018") (footprint "tauntek-hat:USB_C_Receptacle_HRO_TYPE-C-31-M-12_NO_SBU")
+      (reference "J3") (unit 1) (value "USB-TYPE-C-018") (footprint "tauntek-hat:USB_C_Receptacle_HRO_TYPE-C-31-M-12_NO_SBU_CircularHoles")
     )
     (path "/2feda297-9856-40c7-a6de-26ef5c4b169a/a1bc22c6-af81-41fb-82a1-1e00329f20c2"
@@
     )
     (path "/65574413-1451-412e-8903-317c9cabfa8b/646faf83-3b06-4373-950e-0bca5d9259f6"
-      (reference "SW4") (unit 1) (value "EC11x_Encoder") (footprint "Rotary_Encoder:RotaryEncoder_Alps_EC11E-Switch_Vertical_H20mm")
+      (reference "SW4") (unit 1) (value "EC11x_Encoder") (footprint "Rotary_Encoder:RotaryEncoder_Alps_EC11E-Switch_Vertical_H20mm_CircularMountingHoles")
     )
     (path "/75af3154-0603-4d23-93ae-15532c09b444"
@@
     )
     (path "/7e440350-3b06-46cd-b195-35971d0f95cd"
-      (reference "U3") (unit 1) (value "AVR128DB64-IMR") (footprint "Package_DFN_QFN:QFN-64-1EP_9x9mm_P0.5mm_EP7.15x7.15mm_ThermalVias")
+      (reference "U3") (unit 1) (value "AVR128DB64-IMR") (footprint "Package_DFN_QFN:QFN-64-1EP_9x9mm_P0.5mm_EP7.15x7.15mm")
     )
     (path "/e10271d7-3f19-468d-ac2e-d112f94b8b42/624e5576-f377-4f78-ba49-5f8c17c26fc5"
