File: usb.kicad_sch (KiCad schematic)
At the start: 20 parts, among them J3 USB-TYPE-C-018, Q5 NCE30P12S, Q6 DMG2302U, Q7 DMG2302U, U4 CH224K, U5 CH340E

Commit message: Modified PCB for Aisler budget tier
Parts:
- J3: footprint tauntek-hat:USB_C_Receptacle_HRO_TYPE-C-31-M-12_NO_SBU -> (none)
Changed lines of the file:
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@@
     (property "Reference" "J3" (id 0) (at 34.29 34.29 0))
     (property "Value" "USB-TYPE-C-018" (id 1) (at 34.29 36.83 0))
-    (property "Footprint" "tauntek-hat:USB_C_Receptacle_HRO_TYPE-C-31-M-12_NO_SBU" (id 2) (at 38.1 57.15 0)
+    (property "Footprint" "" (id 2) (at 38.1 57.15 0)
       (effects (font (size 1.27 1.27)) hide)
     )
